File: VoidCIC.kicad_sch (KiCad schematic)
At the start: 4 parts, among them U1 SN74LVC1GU04DBVR

Commit message: MAJOR FIX: Repair Schematic to actually be correct now, Redherring32's schematic was a nightmare so I double checked the board and noticed this issue.
Connections:
- net GND: no longer U1.2 (A)
- net RST IN: now also U1.2 (A)
Other:
- moved on the sheet: R1

Commit message: update pcb and sch locations
Other:
- moved on the sheet: C1, R1, U1, VoidCIC1
